Commit message: Added gazebo diffdrive plugin to robot description.

File: src/diffbot_description/urdf/diffbot.urdf.xacro (robot description, xacro)
@@ -14,4 +14,5 @@
 		<xacro:property name="caster_radius" value="0.02"/>
 		<xacro:property name="caster_mass" value="0.1"/>
+		<xacro:property name="update_rate" value="50.0"/>
 		<!-- Linkler -->
 		<link name="base_footprint"/>
@@ -142,3 +143,21 @@
 			<material>Gazebo/Grey</material>
 		</gazebo>
+		<!-- Gazebo Differential Drive Plugini -->
+		<gazebo>
+			<plugin name="diff_drive" filename="libgazebo_ros_diff_drive.so">
+				<ros>
+					<namespace>/</namespace>
+				</ros>
+				<left_joint>left_wheel_joint</left_joint>
+				<right_joint>right_wheel_joint</right_joint>
+				<wheel_separation>${wheel_separation}</wheel_separation>
+				<wheel_diameter>${wheel_radius * 2}</wheel_diameter>
+				<command_topic>cmd_vel</command_topic>
+				<publish_odom>true</publish_odom>
+				<publish_odom_tf>true</publish_odom_tf>
+				<odometry_frame>odom</odometry_frame>
+				<robot_base_frame>base_footprint</robot_base_frame>
+				<update_rate>${update_rate}</update_rate>
+			</plugin>
+		</gazebo>
 </robot>

Commit message: Changed origin z value in base_link from 0 to 0.03

File: src/diffbot_description/urdf/diffbot.urdf.xacro (robot description, xacro)
@@ -19,5 +19,5 @@
 		<link name="base_link">
 			<visual>
-				<origin xyz="0 0 0" rpy="0 0 0"/>
+				<origin xyz="0 0 0.03" rpy="0 0 0"/>
 				<geometry>
 					<box size="${base_length} ${base_width} ${base_height}"/>
@@ -28,5 +28,5 @@
 			</visual>
 			<collision>
-				<origin xyz="0 0 0" rpy="0 0 0"/>
+				<origin xyz="0 0 0.03" rpy="0 0 0"/>
 				<geometry>
 					<box size="${base_length} ${base_width} ${base_height}"/>
@@ -34,5 +34,5 @@
 			</collision>
 			<inertial>
-				<origin xyz="0 0 0" rpy="0 0 0"/>
+				<origin xyz="0 0 0.03" rpy="0 0 0"/>
 				<mass value="${base_mass}"/>
 				<inertia ixx="0.00417" ixy="0" ixz="0" iyy="0.00833" iyz="0" izz="0.01083"/>
